Commit message: Contact sensor topic found, everything works

File: gz_ros2_control_demos/urdf/test_contact_sensor.xacro.urdf (robot description, URDF)
Before this commit: robot diff_drive, 3 links, 2 joints
Joints:
- joint base_sphere_joint: origin xyz=0.0 0.0 10.0 rpy=0 0 0 -> xyz=0.0 0.0 100.0 rpy=0 0 0

Commit message: Add contact sensor force/torque extension and update world file

File: gz_ros2_control_demos/urdf/test_contact_sensor.xacro.urdf (robot description, URDF)
Before this commit: robot diff_drive, 3 links, 2 joints
Joints:
- joint base_sphere_joint: origin xyz=0.0 0.0 100.0 rpy=0 0 0 -> xyz=0.0 0.0 5.0 rpy=0 0 0
